Commit message: changes in xacros

File: src/robot_descriptor/descriptor/camera.xacro (robot description, xacro)
@@ -1,65 +1,19 @@
 <?xml version="1.0"?>
 <robot xmlns:xacro="http://www.ros.org/wiki/xacro">
-    <!-- RGB CAMERA -->
-    <joint name="camera_rgb_joint" type="fixed">
+    <!-- DEPTH CAMERA -->
+    <joint name="camera_joint" type="fixed">
         <parent link="chassis"/>
-        <child link="camera_rgb_link"/>
-        <origin xyz="0.140 -0.03 0.040" rpy="0 0 0"/>
+        <child link="camera_link"/>
+        <origin xyz="0.11 0.0105 0.1285" rpy="0 0 0"/>
     </joint>
-    <link name="camera_rgb_link">
+    <link name="camera_link">
         <visual>
-            <origin xyz="-0.144 0.032 -0.04"
-                    rpy="${-pi/2} ${-pi} ${-pi/2}"/>
+            <origin xyz="0.0 -0.013 0.0" rpy="${pi/2} ${0} ${pi/2}"/>
             <geometry>
-                <mesh filename="package://robot_descriptor/meshes/camera3.stl"
+                <mesh filename="package://robot_descriptor/meshes/IntelRealsense_D435i.stl"
                       scale="0.001 0.001 0.001"/>
-            </geometry>
-            <material name="green"/>
+           </geometry>
+            <material name="grey"/>
         </visual>
     </link>
-    <!-- Optical frame (ROS camera convention) -->
-    <joint name="camera_rgb_optical_joint" type="fixed">
-        <parent link="camera_rgb_link"/>
-        <child link="camera_rgb_optical_link"/>
-        <origin xyz="0 0 -0.008"
-                rpy="${-pi/2} 0 ${-pi/2}"/>
-    </joint>
-    <link name="camera_rgb_optical_link"/>
-    <!-- Gazebo camera sensor -->
-    <gazebo reference="camera_rgb_link">
-        <self_collide>false</self_collide>
-        <material>Gazebo/Green</material>
-        <preserveFixedJoint>true</preserveFixedJoint>
-        <sensor name="modul3_wide" type="camera">
-            <pose>0 0 0 0 0 0</pose>
-            <always_on>true</always_on>
-            <update_rate>30</update_rate>
-            <visualize>true</visualize>
-            <camera>
-                <camera_info_topic>/camera/rgb/camera_info</camera_info_topic>
-                <horizontal_fov>1.78</horizontal_fov>
-                <image>
-                    <width>640</width>
-                    <height>480</height>
-                    <format>R8G8B8</format>
-                </image>
-                <clip>
-                    <near>0.05</near>
-                    <far>8.0</far>
-                </clip>
-                <distortion>
-                    <k1>-0.02</k1>
-                    <k2>0.01</k2>
-                    <k3>0.0</k3>
-                    <p1>0.0</p1>
-                    <p2>0.0</p2>
-                </distortion>
-                <!-- CHANGED: aggiunto optical_frame_id -->
-                <optical_frame_id>camera_rgb_optical_link</optical_frame_id>
-            </camera>
-            <topic>camera/rgb/image_raw</topic>
-            <!-- REMOVED: questa riga rompeva l'orientazione -->
-            <!-- <gz_frame_id>camera_rgb_optical_link</gz_frame_id> -->
-        </sensor>
-    </gazebo>
 </robot>

File: src/robot_descriptor/descriptor/robot.urdf.xacro (robot description, xacro)
@@ -5,6 +5,5 @@
     <xacro:include filename="robot_core.xacro" />
     <xacro:include filename="lidar.xacro" />
-      <!-- <xacro:include filename="camera.xacro" /> -->
-    <xacro:include filename="depth_camera.xacro" />
+    <xacro:include filename="camera.xacro" />
     <xacro:if value="$(arg use_sim_camera)">
         <!--<xacro:include filename="camera_frames.xacro"/>-->

Commit message: fix name link

File: src/robot_descriptor/descriptor/camera.xacro (robot description, xacro)
@@ -7,5 +7,5 @@
         <origin xyz="0.11 0.0105 0.1285" rpy="0 0 0"/>
     </joint>
-    <link name="camera_link">
+    <link name="realsense_link">
         <visual>
             <origin xyz="0.0 -0.013 0.0" rpy="${pi/2} ${0} ${pi/2}"/>

File: src/robot_descriptor/descriptor/camera_frames.xacro (robot description, xacro)
@@ -18,5 +18,5 @@
   <link name="camera_color_optical_frame"/>
   <!-- Gazebo RGBD camera sensor -->
-  <gazebo reference="camera_link">
+  <gazebo reference="realsense_link">
     <preserveFixedJoint>true</preserveFixedJoint>
     <self_collide>false</self_collide>
@@ -39,5 +39,5 @@
         </clip>
         <!-- ROS optical frame -->
-        <optical_frame_id>camera_link</optical_frame_id>
+        <optical_frame_id>realsense_link</optical_frame_id>
       </camera>
       <camera_info_topic>camera/rgbd/camera_info</camera_info_topic>

Commit message: fix camera tf

File: src/robot_descriptor/descriptor/camera.xacro (robot description, xacro)
@@ -4,5 +4,5 @@
     <joint name="camera_joint" type="fixed">
         <parent link="chassis"/>
-        <child link="camera_link"/>
+        <child link="realsense_link"/>
         <origin xyz="0.11 0.0105 0.1285" rpy="0 0 0"/>
     </joint>

Commit message: Add SLAM module and update robot configuration

File: src/robot_descriptor/descriptor/camera.xacro (robot description, xacro)
@@ -2,5 +2,5 @@
 <robot xmlns:xacro="http://www.ros.org/wiki/xacro">
     <!-- DEPTH CAMERA -->
-    <joint name="camera_joint" type="fixed">
+    <joint name="realsense_joint" type="fixed">
         <parent link="chassis"/>
         <child link="realsense_link"/>
@@ -17,3 +17,10 @@
         </visual>
     </link>
+    <joint name="camera_joint" type="fixed">
+        <parent link="realsense_link"/>
+        <child link="camera_link"/>
+        <origin xyz="0.0 0.0 0.0" rpy="0 0 0"/>
+    </joint>
+    <link name="camera_link">
+    </link>
 </robot>
